File: XBee.kicad_sch (KiCad schematic)
At the start: 0 parts

Commit message: xbee initial addition
Parts:
- added IC1: XBP9B-DMST-002, UTSVT_ICs:XBP9B-DMST-002, symbol utsvt-chips:XBP9B-DMST-002
Changed lines of the file:
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@@
 (kicad_sch (version 20230121) (generator eeschema)
   (paper "A4")
+  (symbol (lib_id "utsvt-chips:XBP9B-DMST-002") (at 134.62 86.36 0) (unit 1)
+    (in_bom yes) (on_board yes) (dnp no) (fields_autoplaced)
+    (property "Reference" "IC1" (at 146.05 78.74 0)
+      (effects (font (size 1.27 1.27)))
+    )
+    (property "Value" "XBP9B-DMST-002" (at 146.05 81.28 0)
+      (effects (font (size 1.27 1.27)))
+    )
+    (property "Footprint" "UTSVT_ICs:XBP9B-DMST-002" (at 153.67 181.28 0)
+      (effects (font (size 1.27 1.27)) (justify left top) hide)
+    )
+    (property "Datasheet" "https://componentsearchengine.com/Datasheets/1/XBP9B-DMST-002.pdf" (at 153.67 281.28 0)
+      (effects (font (size 1.27 1.27)) (justify left top) hide)
+    )
+    (property "Height" "" (at 153.67 481.28 0)
+      (effects (font (size 1.27 1.27)) (justify left top) hide)
+    )
+    (property "Mouser Part Number" "888-XBP9B-DMST-002" (at 153.67 581.28 0)
+      (effects (font (size 1.27 1.27)) (justify left top) hide)
+    )
+    (property "Mouser Price/Stock" "https://www.mouser.com/Search/Refine.aspx?Keyword=888-XBP9B-DMST-002" (at 153.67 681.28 0)
+      (effects (font (size 1.27 1.27)) (justify left top) hide)
+    )
+    (property "Manufacturer_Name" "Digi International" (at 153.67 781.28 0)
+      (effects (font (size 1.27 1.27)) (justify left top) hide)
+    )
+    (property "Manufacturer_Part_Number" "XBP9B-DMST-002" (at 153.67 881.28 0)
+      (effects (font (size 1.27 1.27)) (justify left top) hide)
+    )
+    (pin "1")
+    (pin "10")
+    (pin "11")
+    (pin "12")
+    (pin "13")
+    (pin "14")
+    (pin "15")
+    (pin "16")
+    (pin "17")
+    (pin "18")
+    (pin "19")
+    (pin "2")
+    (pin "20")
+    (pin "3")
+    (pin "4")
+    (pin "5")
+    (pin "6")
+    (pin "7")
+    (pin "8")
+    (pin "9")
+    (instances
+      (project "Telemetry-LeaderDaughterboard"
+        (path "/68339661-e19b-41cd-88a0-173b08fffb74/10d4909c-7335-4443-82bb-ba70347b7795"
+          (reference "IC1") (unit 1)
+        )
+      )
+    )
+  )
 )
